Commit message: dual robot Universal updated

File: dual_arm_robot_description/robot/dual_ur_robotiq.urdf.xacro (robot description, xacro)
@@ -2,5 +2,6 @@
 <robot xmlns:xacro="http://wiki.ros.org/xacro" name="dual_ur_robotiq">
   <xacro:property name="PI" value="3.1415926535897931"/>
-  <xacro:arg name="transmission_hw_interface" default="hardware_interface/PositionJointInterface"/>
+  <!-- ur5e -->
+  <xacro:include filename="$(find dual_arm_robot_description)/robot/ur5e.urdf.xacro" />
   <link name="world"/>
   <!-- Stand -->
@@ -14,5 +15,5 @@
       <origin xyz="0 0 0" rpy="0 0 3.1416"/>
       <geometry>
-        <mesh filename="package://dual_ur_robotiq_description/meshes/dual_arm_mount.STL" scale="0.001 0.001 0.001" />
+        <mesh filename="package://dual_arm_robot_description/meshes/dual_arm_mount.STL" scale="0.001 0.001 0.001" />
       </geometry>
       <material name="DarkGrey">
@@ -23,5 +24,5 @@
       <origin xyz="0 0 0" rpy="0 0 3.1416"/>
       <geometry>
-        <mesh filename="package://dual_ur_robotiq_description/meshes/dual_arm_mount.STL" scale="0.001 0.001 0.001" />
+        <mesh filename="package://dual_arm_robot_description/meshes/dual_arm_mount.STL" scale="0.001 0.001 0.001" />
       </geometry>
     </collision>
@@ -34,13 +35,7 @@
     <child link="stand"/>
   </joint>
-<!-- (1) UR5 (extracted from "ur_description/ur5_upload.launch" from "universal_robot" package-->
-  <!-- common stuff -->
-  <xacro:include filename="$(find dual_ur_robotiq_description)/urdf/common.gazebo.xacro" />
-  <!-- ur5e -->
-  <xacro:include filename="$(find dual_ur_robotiq_description)/urdf/ur5e.urdf.xacro" />
-  <!-- left arm -->
-  <xacro:ur5e_robot prefix="left_" joint_limited="false" transmission_hw_interface="$(arg transmission_hw_interface)"/>
-  <!-- right arm -->
-  <xacro:ur5e_robot prefix="right_" joint_limited="false" transmission_hw_interface="$(arg transmission_hw_interface)"/>
+  <!-- Spawn 2 UR5e arms -->
+  <xacro:ur5e_robot prefix="left_" joint_limited="false" />
+  <xacro:ur5e_robot prefix="right_" joint_limited="false" />
   <joint name="left_arm_joint" type="fixed">
     <parent link="stand" />
@@ -53,3 +48,10 @@
     <origin xyz="0 -0.23412 0.50271" rpy="-3.1416 0.610865 1.5708" />
   </joint>
+<!-- (1) UR5 (extracted from "ur_description/ur5_upload.launch" from "universal_robot" package-->
+  <!-- common stuff -->
+  <!-- <xacro:include filename="$(find dual_arm_robot_description)/urdf/common.gazebo.xacro" /> -->
+  <!-- left arm -->
+  <!-- <xacro:ur5e_robot prefix="left_" joint_limited="false" transmission_hw_interface="$(arg transmission_hw_interface)"/> -->
+  <!-- right arm -->
+  <!-- <xacro:ur5e_robot prefix="right_" joint_limited="false" transmission_hw_interface="$(arg transmission_hw_interface)"/> -->
 </robot>

File: dual_arm_robot_description/robot/ur5e.urdf.xacro (robot description, xacro)
@@ -1,6 +1,4 @@
 <?xml version="1.0"?>
 <robot xmlns:xacro="http://ros.org/wiki/xacro">
-  <xacro:include filename="$(find dual_ur_robotiq_description)/urdf/ur.transmission.xacro" />
-  <xacro:include filename="$(find dual_ur_robotiq_description)/urdf/ur.gazebo.xacro" />
   <xacro:macro name="cylinder_inertial" params="radius length mass *origin">
     <inertial>
@@ -88,13 +86,13 @@
       <visual>
         <geometry>
-          <mesh filename="package://dual_ur_robotiq_description/meshes/ur3e/visual/base.dae" />
-        </geometry>
-        <material name="LightGrey">
-          <color rgba="0.7 0.7 0.7 1.0"/>
-        </material>
-      </visual>
-      <collision>
-        <geometry>
-          <mesh filename="package://dual_ur_robotiq_description/meshes/ur3e/collision/base.stl" />
+          <mesh filename="package://dual_arm_robot_description/meshes/ur3e/visual/base.dae" />
+        </geometry>
+        <material name="LightGrey">
+          <color rgba="0.7 0.7 0.7 1.0"/>
+        </material>
+      </visual>
+      <collision>
+        <geometry>
+          <mesh filename="package://dual_arm_robot_description/meshes/ur3e/collision/base.stl" />
         </geometry>
       </collision>
@@ -125,13 +123,13 @@
       <visual>
         <geometry>
-          <mesh filename="package://dual_ur_robotiq_description/meshes/ur3e/visual/shoulder.dae" />
-        </geometry>
-        <material name="LightGrey">
-          <color rgba="0.7 0.7 0.7 1.0"/>
-        </material>
-      </visual>
-      <collision>
-        <geometry>
-          <mesh filename="package://dual_ur_robotiq_description/meshes/ur3e/collision/shoulder.stl" />
+          <mesh filename="package://dual_arm_robot_description/meshes/ur3e/visual/shoulder.dae" />
+        </geometry>
+        <material name="LightGrey">
+          <color rgba="0.7 0.7 0.7 1.0"/>
+        </material>
+      </visual>
+      <collision>
+        <geometry>
+          <mesh filename="package://dual_arm_robot_description/meshes/ur3e/collision/shoulder.stl" />
         </geometry>
       </collision>
@@ -162,13 +160,13 @@
       <visual>
         <geometry>
-          <mesh filename="package://dual_ur_robotiq_description/meshes/ur3e/visual/upperarm.dae" />
-        </geometry>
-        <material name="LightGrey">
-          <color rgba="0.7 0.7 0.7 1.0"/>
-        </material>
-      </visual>
-      <collision>
-        <geometry>
-          <mesh filename="package://dual_ur_robotiq_description/meshes/ur3e/collision/upperarm.stl" />
+          <mesh filename="package://dual_arm_robot_description/meshes/ur3e/visual/upperarm.dae" />
+        </geometry>
+        <material name="LightGrey">
+          <color rgba="0.7 0.7 0.7 1.0"/>
+        </material>
+      </visual>
+      <collision>
+        <geometry>
+          <mesh filename="package://dual_arm_robot_description/meshes/ur3e/collision/upperarm.stl" />
         </geometry>
       </collision>
@@ -199,13 +197,13 @@
       <visual>
         <geometry>
-          <mesh filename="package://dual_ur_robotiq_description/meshes/ur3e/visual/forearm.dae" />
-        </geometry>
-        <material name="LightGrey">
-          <color rgba="0.7 0.7 0.7 1.0"/>
-        </material>
-      </visual>
-      <collision>
-        <geometry>
-          <mesh filename="package://dual_ur_robotiq_description/meshes/ur3e/collision/forearm.stl" />
+          <mesh filename="package://dual_arm_robot_description/meshes/ur3e/visual/forearm.dae" />
+        </geometry>
+        <material name="LightGrey">
+          <color rgba="0.7 0.7 0.7 1.0"/>
+        </material>
+      </visual>
+      <collision>
+        <geometry>
+          <mesh filename="package://dual_arm_robot_description/meshes/ur3e/collision/forearm.stl" />
         </geometry>
       </collision>
@@ -236,13 +234,13 @@
       <visual>
         <geometry>
-          <mesh filename="package://dual_ur_robotiq_description/meshes/ur3e/visual/wrist1.dae" />
-        </geometry>
-        <material name="LightGrey">
-          <color rgba="0.7 0.7 0.7 1.0"/>
-        </material>
-      </visual>
-      <collision>
-        <geometry>
-          <mesh filename="package://dual_ur_robotiq_description/meshes/ur3e/collision/wrist1.stl" />
+          <mesh filename="package://dual_arm_robot_description/meshes/ur3e/visual/wrist1.dae" />
+        </geometry>
+        <material name="LightGrey">
+          <color rgba="0.7 0.7 0.7 1.0"/>
+        </material>
+      </visual>
+      <collision>
+        <geometry>
+          <mesh filename="package://dual_arm_robot_description/meshes/ur3e/collision/wrist1.stl" />
         </geometry>
       </collision>
@@ -273,13 +271,13 @@
       <visual>
         <geometry>
-          <mesh filename="package://dual_ur_robotiq_description/meshes/ur3e/visual/wrist2.dae" />
-        </geometry>
-        <material name="LightGrey">
-          <color rgba="0.7 0.7 0.7 1.0"/>
-        </material>
-      </visual>
-      <collision>
-        <geometry>
-          <mesh filename="package://dual_ur_robotiq_description/meshes/ur3e/collision/wrist2.stl" />
+          <mesh filename="package://dual_arm_robot_description/meshes/ur3e/visual/wrist2.dae" />
+        </geometry>
+        <material name="LightGrey">
+          <color rgba="0.7 0.7 0.7 1.0"/>
+        </material>
+      </visual>
+      <collision>
+        <geometry>
+          <mesh filename="package://dual_arm_robot_description/meshes/ur3e/collision/wrist2.stl" />
         </geometry>
       </collision>
@@ -310,13 +308,13 @@
       <visual>
         <geometry>
-          <mesh filename="package://dual_ur_robotiq_description/meshes/ur3e/visual/wrist3.dae" />
-        </geometry>
-        <material name="LightGrey">
-          <color rgba="0.7 0.7 0.7 1.0"/>
-        </material>
-      </visual>
-      <collision>
-        <geometry>
-          <mesh filename="package://dual_ur_robotiq_description/meshes/ur3e/collision/wrist3.stl" />
+          <mesh filename="package://dual_arm_robot_description/meshes/ur3e/visual/wrist3.dae" />
+        </geometry>
+        <material name="LightGrey">
+          <color rgba="0.7 0.7 0.7 1.0"/>
+        </material>
+      </visual>
+      <collision>
+        <geometry>
+          <mesh filename="package://dual_arm_robot_description/meshes/ur3e/collision/wrist3.stl" />
         </geometry>
       </collision>
@@ -338,6 +336,4 @@
       </collision>
     </link>
-    <xacro:ur_arm_transmission prefix="${prefix}" />
-    <xacro:ur_arm_gazebo prefix="${prefix}" />
     <!-- ROS base_link to UR 'Base' Coordinates transform -->
     <link name="${prefix}base"/>
@@ -365,5 +361,5 @@
         <origin xyz="0.0 0.0 ${-1.0 * gripper_offset}" rpy="0 0 0" />
         <geometry>
-          <mesh filename="package://dual_ur_robotiq_description/meshes/ur3e/visual/basegripper.STL" scale="0.001 0.001 0.001" />
+          <mesh filename="package://dual_arm_robot_description/meshes/ur3e/visual/basegripper.STL" scale="0.001 0.001 0.001" />
         </geometry>
         <material name="">
@@ -374,5 +370,5 @@
         <origin xyz="0.0 0.0 ${-1.0 * gripper_offset}" rpy="0 0 0" />
         <geometry>
-          <mesh filename="package://dual_ur_robotiq_description/meshes/ur3e/collision/basegripper.STL" scale="0.001 0.001 0.001" />
+          <mesh filename="package://dual_arm_robot_description/meshes/ur3e/collision/basegripper.STL" scale="0.001 0.001 0.001" />
         </geometry>
       </collision>
@@ -392,5 +388,5 @@
       <origin xyz="0 0 0" rpy="0 0 0" />
       <geometry>
-        <mesh filename="package://dual_ur_robotiq_description/meshes/ur3e/visual/finger_1.STL" scale="0.001 0.001 0.001" />
+        <mesh filename="package://dual_arm_robot_description/meshes/ur3e/visual/finger_1.STL" scale="0.001 0.001 0.001" />
       </geometry>
       <material
@@ -403,5 +399,5 @@
       <origin xyz="0 0 0" rpy="0 0 0" />
       <geometry>
-        <mesh filename="package://dual_ur_robotiq_description/meshes/ur3e/collision/finger_1.STL" scale="0.001 0.001 0.001" />
+        <mesh filename="package://dual_arm_robot_description/meshes/ur3e/collision/finger_1.STL" scale="0.001 0.001 0.001" />
       </geometry>
     </collision>
@@ -429,5 +425,5 @@
       <origin xyz="0 0 0" rpy="0 0 0" />
       <geometry>
-        <mesh filename="package://dual_ur_robotiq_description/meshes/ur3e/visual/finger_2.STL" scale="0.001 0.001 0.001" />
+        <mesh filename="package://dual_arm_robot_description/meshes/ur3e/visual/finger_2.STL" scale="0.001 0.001 0.001" />
       </geometry>
       <material
@@ -440,5 +436,5 @@
       <origin xyz="0 0 0" rpy="0 0 0" />
       <geometry>
-        <mesh filename="package://dual_ur_robotiq_description/meshes/ur3e/collision/finger_2.STL" scale="0.001 0.001 0.001" />
+        <mesh filename="package://dual_arm_robot_description/meshes/ur3e/collision/finger_2.STL" scale="0.001 0.001 0.001" />
       </geometry>
     </collision>
