Commit message: dual_arm_updated

File: dual_arm_robot_moveit_config/config/dual_ur_robotiq.ros2_control.xacro (robot description, xacro)
@@ -1,124 +1,329 @@
 <?xml version="1.0"?>
 <robot xmlns:xacro="http://www.ros.org/wiki/xacro">
-    <xacro:macro name="dual_ur_robotiq_ros2_control" params="name initial_positions_file">
+    <xacro:macro name="dual_ur_robotiq_ros2_control" params="
+      name
+      initial_positions_file
+      use_fake_hardware:=false
+      sim_gazebo:=false
+      sim_ignition:=false
+      left_robot_ip:= 192.168.3.212
+      right_robot_ip:= 192.168.3.213
+      reverse_ip:=0.0.0.0
+      left_tf_prefix:=left_
+      right_tf_prefix:=right_
+      script_filename:=/tmp/ur_script.script
+      output_recipe_filename:=/tmp/rtde_output_recipe.txt
+      input_recipe_filename:=/tmp/rtde_input_recipe.txt
+      headless_mode:=false
+      reverse_port:=50001
+      script_sender_port:=50002
+      script_command_port:=50004
+      trajectory_port:=50003
+      use_tool_communication:=false
+      tool_voltage:=0
+      tool_parity:=0
+      tool_baud_rate:=115200
+      tool_stop_bits:=1
+      tool_rx_idle_chars:=1.5
+      tool_tx_idle_chars:=3.5
+      tool_device_name:=/tmp/ttyUR
+      tool_tcp_port:=54321
+      keep_alive_count:=2
+      hash_kinematics:=0">
         <xacro:property name="initial_positions" value="${load_yaml(initial_positions_file)['initial_positions']}"/>
-        <ros2_control name="${name}" type="system">
+        <!-- Left Arm ros2_control -->
+        <ros2_control name="${name}_left_arm" type="system">
             <hardware>
-                <!-- By default, set up controllers for simulation. This won't work on real hardware -->
-                <plugin>mock_components/GenericSystem</plugin>
+                <xacro:if value="${sim_gazebo}">
+                    <plugin>gazebo_ros2_control/GazeboSystem</plugin>
+                </xacro:if>
+                <xacro:if value="${sim_ignition}">
+                    <plugin>ign_ros2_control/IgnitionSystem</plugin>
+                </xacro:if>
+                <xacro:if value="${use_fake_hardware}">
+                    <plugin>mock_components/GenericSystem</plugin>
+                    <param name="fake_sensor_commands">false</param>
+                    <param name="state_following_offset">0.0</param>
+                    <param name="calculate_dynamics">true</param>
+                </xacro:if>
+                <xacro:unless value="${use_fake_hardware or sim_gazebo or sim_ignition}">
+                    <plugin>ur_robot_driver/URPositionHardwareInterface</plugin>
+                    <param name="robot_ip">${left_robot_ip}</param>
+                    <param name="script_filename">${script_filename}</param>
+                    <param name="output_recipe_filename">${output_recipe_filename}</param>
+                    <param name="input_recipe_filename">${input_recipe_filename}</param>
+                    <param name="headless_mode">${headless_mode}</param>
+                    <param name="reverse_port">${reverse_port}</param>
+                    <param name="script_sender_port">${script_sender_port}</param>
+                    <param name="reverse_ip">${reverse_ip}</param>
+                    <param name="script_command_port">${script_command_port}</param>
+                    <param name="trajectory_port">${trajectory_port}</param>
+                    <param name="tf_prefix">${left_tf_prefix}</param>
+                    <param name="non_blocking_read">true</param>
+                    <param name="servoj_gain">2000</param>
+                    <param name="servoj_lookahead_time">0.03</param>
+                    <param name="use_tool_communication">${use_tool_communication}</param>
+                    <param name="kinematics/hash">${hash_kinematics}</param>
+                    <param name="tool_voltage">${tool_voltage}</param>
+                    <param name="tool_parity">${tool_parity}</param>
+                    <param name="tool_baud_rate">${tool_baud_rate}</param>
+                    <param name="tool_stop_bits">${tool_stop_bits}</param>
+                    <param name="tool_rx_idle_chars">${tool_rx_idle_chars}</param>
+                    <param name="tool_tx_idle_chars">${tool_tx_idle_chars}</param>
+                    <param name="tool_device_name">${tool_device_name}</param>
+                    <param name="tool_tcp_port">${tool_tcp_port}</param>
+                    <param name="keep_alive_count">${keep_alive_count}</param>
+                </xacro:unless>
             </hardware>
-            <joint name="left_shoulder_pan_joint">
-                <command_interface name="position"/>
-                <state_interface name="position">
-                  <param name="initial_value">${initial_positions['left_shoulder_pan_joint']}</param>
-                </state_interface>
-                <state_interface name="velocity"/>
-            </joint>
-            <joint name="left_shoulder_lift_joint">
-                <command_interface name="position"/>
-                <state_interface name="position">
-                  <param name="initial_value">${initial_positions['left_shoulder_lift_joint']}</param>
-                </state_interface>
-                <state_interface name="velocity"/>
-            </joint>
-            <joint name="left_elbow_joint">
-                <command_interface name="position"/>
-                <state_interface name="position">
-                  <param name="initial_value">${initial_positions['left_elbow_joint']}</param>
-                </state_interface>
-                <state_interface name="velocity"/>
-            </joint>
-            <joint name="left_wrist_1_joint">
-                <command_interface name="position"/>
-                <state_interface name="position">
-                  <param name="initial_value">${initial_positions['left_wrist_1_joint']}</param>
-                </state_interface>
-                <state_interface name="velocity"/>
-            </joint>
-            <joint name="left_wrist_2_joint">
-                <command_interface name="position"/>
-                <state_interface name="position">
-                  <param name="initial_value">${initial_positions['left_wrist_2_joint']}</param>
-                </state_interface>
-                <state_interface name="velocity"/>
-            </joint>
-            <joint name="left_wrist_3_joint">
-                <command_interface name="position"/>
-                <state_interface name="position">
-                  <param name="initial_value">${initial_positions['left_wrist_3_joint']}</param>
-                </state_interface>
-                <state_interface name="velocity"/>
-            </joint>
-            <joint name="right_shoulder_pan_joint">
-                <command_interface name="position"/>
-                <state_interface name="position">
-                  <param name="initial_value">${initial_positions['right_shoulder_pan_joint']}</param>
-                </state_interface>
-                <state_interface name="velocity"/>
-            </joint>
-            <joint name="right_shoulder_lift_joint">
-                <command_interface name="position"/>
-                <state_interface name="position">
-                  <param name="initial_value">${initial_positions['right_shoulder_lift_joint']}</param>
-                </state_interface>
-                <state_interface name="velocity"/>
-            </joint>
-            <joint name="right_elbow_joint">
-                <command_interface name="position"/>
-                <state_interface name="position">
-                  <param name="initial_value">${initial_positions['right_elbow_joint']}</param>
-                </state_interface>
-                <state_interface name="velocity"/>
-            </joint>
-            <joint name="right_wrist_1_joint">
-                <command_interface name="position"/>
-                <state_interface name="position">
-                  <param name="initial_value">${initial_positions['right_wrist_1_joint']}</param>
-                </state_interface>
-                <state_interface name="velocity"/>
-            </joint>
-            <joint name="right_wrist_2_joint">
-                <command_interface name="position"/>
-                <state_interface name="position">
-                  <param name="initial_value">${initial_positions['right_wrist_2_joint']}</param>
-                </state_interface>
-                <state_interface name="velocity"/>
-            </joint>
-            <joint name="right_wrist_3_joint">
-                <command_interface name="position"/>
-                <state_interface name="position">
-                  <param name="initial_value">${initial_positions['right_wrist_3_joint']}</param>
-                </state_interface>
-                <state_interface name="velocity"/>
-            </joint>
-            <joint name="left_joint_finger_1">
-                <command_interface name="position"/>
-                <state_interface name="position">
-                  <param name="initial_value">${initial_positions['left_joint_finger_1']}</param>
-                </state_interface>
-                <state_interface name="velocity"/>
-            </joint>
-            <joint name="left_joint_finger_2">
-                <command_interface name="position"/>
-                <state_interface name="position">
-                  <param name="initial_value">${initial_positions['left_joint_finger_2']}</param>
-                </state_interface>
-                <state_interface name="velocity"/>
-            </joint>
-            <joint name="right_joint_finger_1">
-                <command_interface name="position"/>
-                <state_interface name="position">
-                  <param name="initial_value">${initial_positions['right_joint_finger_1']}</param>
-                </state_interface>
-                <state_interface name="velocity"/>
-            </joint>
-            <joint name="right_joint_finger_2">
-                <command_interface name="position"/>
-                <state_interface name="position">
-                  <param name="initial_value">${initial_positions['right_joint_finger_2']}</param>
-                </state_interface>
-                <state_interface name="velocity"/>
-            </joint>
+            <joint name="${left_tf_prefix}shoulder_pan_joint">
+                <command_interface name="position"/>
+                <command_interface name="velocity"/>
+                <state_interface name="position">
+                    <param name="initial_value">${initial_positions['left_shoulder_pan_joint']}</param>
+                </state_interface>
+                <state_interface name="velocity"/>
+                <state_interface name="effort"/>
+            </joint>
+            <joint name="${left_tf_prefix}shoulder_lift_joint">
+                <command_interface name="position"/>
+                <command_interface name="velocity"/>
+                <state_interface name="position">
+                    <param name="initial_value">${initial_positions['left_shoulder_lift_joint']}</param>
+                </state_interface>
+                <state_interface name="velocity"/>
+                <state_interface name="effort"/>
+            </joint>
+            <joint name="${left_tf_prefix}elbow_joint">
+                <command_interface name="position"/>
+                <command_interface name="velocity"/>
+                <state_interface name="position">
+                    <param name="initial_value">${initial_positions['left_elbow_joint']}</param>
+                </state_interface>
+                <state_interface name="velocity"/>
+                <state_interface name="effort"/>
+            </joint>
+            <joint name="${left_tf_prefix}wrist_1_joint">
+                <command_interface name="position"/>
+                <command_interface name="velocity"/>
+                <state_interface name="position">
+                    <param name="initial_value">${initial_positions['left_wrist_1_joint']}</param>
+                </state_interface>
+                <state_interface name="velocity"/>
+                <state_interface name="effort"/>
+            </joint>
+            <joint name="${left_tf_prefix}wrist_2_joint">
+                <command_interface name="position"/>
+                <command_interface name="velocity"/>
+                <state_interface name="position">
+                    <param name="initial_value">${initial_positions['left_wrist_2_joint']}</param>
+                </state_interface>
+                <state_interface name="velocity"/>
+                <state_interface name="effort"/>
+            </joint>
+            <joint name="${left_tf_prefix}wrist_3_joint">
+                <command_interface name="position"/>
+                <command_interface name="velocity"/>
+                <state_interface name="position">
+                    <param name="initial_value">${initial_positions['left_wrist_3_joint']}</param>
+                </state_interface>
+                <state_interface name="velocity"/>
+                <state_interface name="effort"/>
+            </joint>
+            <xacro:unless value="${sim_gazebo or sim_ignition}">
+                <sensor name="${left_tf_prefix}tcp_fts_sensor">
+                    <state_interface name="force.x"/>
+                    <state_interface name="force.y"/>
+                    <state_interface name="force.z"/>
+                    <state_interface name="torque.x"/>
+                    <state_interface name="torque.y"/>
+                    <state_interface name="torque.z"/>
+                </sensor>
+                <sensor name="${left_tf_prefix}tcp_pose">
+                    <state_interface name="position.x"/>
+                    <state_interface name="position.y"/>
+                    <state_interface name="position.z"/>
+                    <state_interface name="orientation.x"/>
+                    <state_interface name="orientation.y"/>
+                    <state_interface name="orientation.z"/>
+                    <state_interface name="orientation.w"/>
+                </sensor>
+            </xacro:unless>
         </ros2_control>
+        <!-- Right Arm ros2_control -->
+        <ros2_control name="${name}_right_arm" type="system">
+            <hardware>
+                <xacro:if value="${sim_gazebo}">
+                    <plugin>gazebo_ros2_control/GazeboSystem</plugin>
+                </xacro:if>
+                <xacro:if value="${sim_ignition}">
+                    <plugin>ign_ros2_control/IgnitionSystem</plugin>
+                </xacro:if>
+                <xacro:if value="${use_fake_hardware}">
+                    <plugin>mock_components/GenericSystem</plugin>
+                    <param name="fake_sensor_commands">false</param>
+                    <param name="state_following_offset">0.0</param>
+                    <param name="calculate_dynamics">true</param>
+                </xacro:if>
+                <xacro:unless value="${use_fake_hardware or sim_gazebo or sim_ignition}">
+                    <plugin>ur_robot_driver/URPositionHardwareInterface</plugin>
+                    <param name="robot_ip">${right_robot_ip}</param>
+                    <param name="script_filename">${script_filename}</param>
+                    <param name="output_recipe_filename">${output_recipe_filename}</param>
+                    <param name="input_recipe_filename">${input_recipe_filename}</param>
+                    <param name="headless_mode">${headless_mode}</param>
+                    <param name="reverse_port">${reverse_port}</param>
+                    <param name="script_sender_port">${script_sender_port}</param>
+                    <param name="reverse_ip">${reverse_ip}</param>
+                    <param name="script_command_port">${script_command_port}</param>
+                    <param name="trajectory_port">${trajectory_port}</param>
+                    <param name="tf_prefix">${right_tf_prefix}</param>
+                    <param name="non_blocking_read">true</param>
+                    <param name="servoj_gain">2000</param>
+                    <param name="servoj_lookahead_time">0.03</param>
+                    <param name="use_tool_communication">${use_tool_communication}</param>
+                    <param name="kinematics/hash">${hash_kinematics}</param>
+                    <param name="tool_voltage">${tool_voltage}</param>
+                    <param name="tool_parity">${tool_parity}</param>
+                    <param name="tool_baud_rate">${tool_baud_rate}</param>
+                    <param name="tool_stop_bits">${tool_stop_bits}</param>
+                    <param name="tool_rx_idle_chars">${tool_rx_idle_chars}</param>
+                    <param name="tool_tx_idle_chars">${tool_tx_idle_chars}</param>
+                    <param name="tool_device_name">${tool_device_name}</param>
+                    <param name="tool_tcp_port">${tool_tcp_port}</param>
+                    <param name="keep_alive_count">${keep_alive_count}</param>
+                </xacro:unless>
+            </hardware>
+            <joint name="${right_tf_prefix}shoulder_pan_joint">
+                <command_interface name="position"/>
+                <command_interface name="velocity"/>
+                <state_interface name="position">
+                    <param name="initial_value">${initial_positions['right_shoulder_pan_joint']}</param>
+                </state_interface>
+                <state_interface name="velocity"/>
+                <state_interface name="effort"/>
+            </joint>
+            <joint name="${right_tf_prefix}shoulder_lift_joint">
+                <command_interface name="position"/>
+                <command_interface name="velocity"/>
+                <state_interface name="position">
+                    <param name="initial_value">${initial_positions['right_shoulder_lift_joint']}</param>
+                </state_interface>
+                <state_interface name="velocity"/>
+                <state_interface name="effort"/>
+            </joint>
+            <joint name="${right_tf_prefix}elbow_joint">
+                <command_interface name="position"/>
+                <command_interface name="velocity"/>
+                <state_interface name="position">
+                    <param name="initial_value">${initial_positions['right_elbow_joint']}</param>
+                </state_interface>
+                <state_interface name="velocity"/>
+                <state_interface name="effort"/>
+            </joint>
+            <joint name="${right_tf_prefix}wrist_1_joint">
+                <command_interface name="position"/>
+                <command_interface name="velocity"/>
+                <state_interface name="position">
+                    <param name="initial_value">${initial_positions['right_wrist_1_joint']}</param>
+                </state_interface>
+                <state_interface name="velocity"/>
+                <state_interface name="effort"/>
+            </joint>
+            <joint name="${right_tf_prefix}wrist_2_joint">
+                <command_interface name="position"/>
+                <command_interface name="velocity"/>
+                <state_interface name="position">
+                    <param name="initial_value">${initial_positions['right_wrist_2_joint']}</param>
+                </state_interface>
+                <state_interface name="velocity"/>
+                <state_interface name="effort"/>
+            </joint>
+            <joint name="${right_tf_prefix}wrist_3_joint">
+                <command_interface name="position"/>
+                <command_interface name="velocity"/>
+                <state_interface name="position">
+                    <param name="initial_value">${initial_positions['right_wrist_3_joint']}</param>
+                </state_interface>
+                <state_interface name="velocity"/>
+                <state_interface name="effort"/>
+            </joint>
+            <xacro:unless value="${sim_gazebo or sim_ignition}">
+                <sensor name="${right_tf_prefix}tcp_fts_sensor">
+                    <state_interface name="force.x"/>
+                    <state_interface name="force.y"/>
+                    <state_interface name="force.z"/>
+                    <state_interface name="torque.x"/>
+                    <state_interface name="torque.y"/>
+                    <state_interface name="torque.z"/>
+                </sensor>
+                <sensor name="${right_tf_prefix}tcp_pose">
+                    <state_interface name="position.x"/>
+                    <state_interface name="position.y"/>
+                    <state_interface name="position.z"/>
+                    <state_interface name="orientation.x"/>
+                    <state_interface name="orientation.y"/>
+                    <state_interface name="orientation.z"/>
+                    <state_interface name="orientation.w"/>
+                </sensor>
+            </xacro:unless>
+        </ros2_control>
+        <!-- Left Gripper ros2_control -->
+        <!-- <ros2_control name="${name}_left_gripper" type="system">
+            <hardware>
+                <xacro:if value="${use_fake_hardware}">
+                    <plugin>mock_components/GenericSystem</plugin>
+                </xacro:if>
+                <xacro:unless value="${use_fake_hardware}">
+                    <plugin>robotiq_controllers/Robotiq2FGripperHardwareInterface</plugin>
+                    <param name="robot_ip">${left_robot_ip}</param>
+                    <param name="tool_device_name">${tool_device_name}</param>
+                    <param name="tool_tcp_port">${tool_tcp_port}</param>
+                    <param name="use_tool_communication">true</param>
+                </xacro:unless>
+            </hardware>
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
File: dual_arm_robot_moveit_config/config/dual_ur_robotiq.urdf.xacro (robot description, xacro)
@@ -6,4 +6,4 @@
     <!-- Import control_xacro -->
     <xacro:include filename="dual_ur_robotiq.ros2_control.xacro" />
-    <xacro:dual_ur_robotiq_ros2_control name="FakeSystem" initial_positions_file="$(arg initial_positions_file)"/>
+    <!-- <xacro:dual_ur_robotiq_ros2_control name="FakeSystem" initial_positions_file="$(arg initial_positions_file)"/> -->
 </robot>
